File: Hardware/XM125_Breakout.sch (EAGLE design)
At the start: 53 parts, among them J13 SWD (DNP), J2 RIGHT_ANGLE, J3 RIGHT_ANGLE, U1 XM125, U2 RT9080-33GJ5, U3 RT9080-18GJ5, U4 CH340C, U5 ESD Diode

Commit message: Cleanup repo; design review changes
Check design review document for full list of changes/details.
Parts:
- removed J10, J11, J12, J9: (no value), SparkFun-Connectors:CONN_01PTH_NO_SILK_STAND
- removed J4: (no value), SparkFun-Connectors:CONN_041X04_NO_SILK
- removed J5, J6: (no value), SparkFun-Connectors:CONN_021X02_NO_SILK
- removed J7: (no value), SparkFun-Connectors:CONN_05NO_SILK
- removed J8: (no value), SparkFun-Connectors:CONN_031X03_NO_SILK
- added J14: (no value), SparkFun-Connectors:CONN_09NO_SILK
- added J15: (no value), SparkFun-Connectors:CONN_111X11_NO_SILK
Connections:
- net !XM125_INT: now also J14.9; no longer J11.1
- net !XM125_RESET: now also J14.1; no longer J9.1
- net 1.8V: now also J14.7; no longer J7.4
- net 3.3V: now also J14.8, J15.4; no longer J4.2, J7.5
- net DEBUG_UART-RX: now also J15.7; no longer J5.1
- net DEBUG_UART-TX: now also J15.8; no longer J5.2
- net GND: now also J14.4, J14.5, J15.5; no longer J4.1, J7.1, J7.2
- net SCL: now also J15.2; no longer J4.4
- net SDA: now also J15.3; no longer J4.3
- net SWD_CLK: now also J14.2; no longer J6.2
- net SWD_IO: now also J14.3; no longer J6.1
- net V_USB: now also J14.6; no longer J7.3
- net WAKE_UP: now also J15.1; no longer J12.1
- net XM125_GPIO0: now also J15.9; no longer J8.1
- net XM125_GPIO1: now also J15.10; no longer J8.2
- net XM125_GPIO2/BOOT0: now also J15.11; no longer J8.3
- net XM125_I2C_ADDRESS: now also J15.6; no longer J10.1
Other:
- note added: "Cut SHLD to disconnect the SHLD from GND"
- note added: "USB-to-Serial Converter CH340C"
- note removed: "USB-to-Serial Converter"
- moved on the sheet: U5
